Commit message: Modify are Made

File: description/so101_new_calib.urdf (robot description, URDF)
Before this commit: robot robot, 8 links, 7 joints
Links:
- link base_link: geometry collision mesh filename=package://tarsarm_sim/description/assets/base_motor_holder_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; collision mesh filename=package://tarsarm_sim/description/assets/base_so101_v2.stl
- link lower_arm_link: geometry collision mesh filename=package://tarsarm_sim/description/assets/motor_holder_so101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; collision mesh filename=package://tarsarm_sim/description/assets/sts3215_03a_v1.stl
- link moving_jaw_so101_v1_link: geometry collision mesh filename=package://tarsarm_sim/description/assets/moving_jaw_so101_v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; visual mesh filename=package://tarsarm_sim/description/assets/moving_jaw_so101_v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

File: description/so101_old_calib.urdf (robot description, URDF)
Before this commit: robot robot, 8 links, 7 joints
Links:
- removed link base_link
- removed link gripper_frame_link
- removed link gripper_link
- removed link lower_arm_link
- removed link moving_jaw_so101_v1_link
- removed link shoulder_link
- removed link upper_arm_link
- removed link wrist_link
- added link base, mass 0.147; collision mesh filename=assets/base_motor_holder_so101_v1.stl; collision mesh filename=assets/base_so101_v2.stl
- added link gripper, mass 0.087; collision mesh filename=assets/sts3215_03a_v1.stl; collision mesh filename=assets/wrist_roll_follower_so101_v1.stl
- added link jaw, mass 0.012; collision mesh filename=assets/moving_jaw_so101_v1.stl; visual mesh filename=assets/moving_jaw_so101_v1.stl
- added link lower_arm, mass 0.104; collision mesh filename=assets/motor_holder_so101_wrist_v1.stl; collision mesh filename=assets/sts3215_03a_v1.stl
- added link shoulder, mass 0.100006; collision mesh filename=assets/motor_holder_so101_base_v1.stl; collision mesh filename=assets/rotation_pitch_so101_v1.stl
- added link upper_arm, mass 0.103; collision mesh filename=assets/sts3215_03a_v1.stl; collision mesh filename=assets/upper_arm_so101_v1.stl
- added link wrist, mass 0.079; collision mesh filename=assets/sts3215_03a_no_horn_v1.stl; collision mesh filename=assets/wrist_roll_pitch_so101_v2.stl
Joints:
- removed joint gripper_frame_joint
- joint elbow_flex: child lower_arm_link -> lower_arm; limit lower=-1.69 upper=1.69 effort=10 velocity=10 -> lower=-0.174533 upper=3.14159 effort=10 velocity=10; origin xyz=-0.11257 -0.028 1.73763e-16 rpy=-3.63608e-16 8.74301e-16 1.5708 -> xyz=-0.028 0.11257 1.24466e-16 rpy=1.89432e-15 -3.22659e-15 -3.14159; parent upper_arm_link -> upper_arm
- joint gripper: child moving_jaw_so101_v1_link -> jaw; origin xyz=0.0202 0.0188 -0.0234 rpy=1.5708 -5.24284e-08 -1.41553e-15 -> xyz=0.0202 0.0188 -0.0234 rpy=1.5708 -7.91661e-17 -1.0396e-16; parent gripper_link -> gripper
- joint shoulder_lift: child upper_arm_link -> upper_arm; limit lower=-1.74533 upper=1.74533 effort=10 velocity=10 -> lower=-3.31613 upper=0.174533 effort=10 velocity=10; origin xyz=-0.0303992 -0.0182778 -0.0542 rpy=-1.5708 -1.5708 0 -> xyz=-0.0303992 -0.0182778 -0.0542 rpy=-1.5708 1.5708 0; parent shoulder_link -> shoulder
- joint shoulder_pan: child shoulder_link -> shoulder; origin xyz=0.0388353 -8.97657e-09 0.0624 rpy=3.14159 4.18253e-17 -3.14159 -> xyz=0.0207909 -0.0230745 0.0948817 rpy=-3.14159 6.03684e-16 1.5708; parent base_link -> base
- joint wrist_flex: child wrist_link -> wrist; origin xyz=-0.1349 0.0052 3.62355e-17 rpy=4.02456e-15 8.67362e-16 -1.5708 -> xyz=-0.0052 -0.1349 3.40439e-16 rpy=-1.41553e-15 4.91611e-15 7.56157e-09; parent lower_arm_link -> lower_arm
- joint wrist_roll: child gripper_link -> gripper; limit lower=-2.74385 upper=2.84121 effort=10 velocity=10 -> lower=-2.79253 upper=2.79253 effort=10 velocity=10; origin xyz=5.55112e-17 -0.0611 0.0181 rpy=1.5708 0.0486795 3.14159 -> xyz=2.77556e-17 -0.0611 0.0181 rpy=1.5708 -9.38083e-08 3.14159; parent wrist_link -> wrist
